File: Add-ons/Power Sandwitch/Power Sandwitch.brd (EAGLE design)
At the start: 16 x 60 mm, 13 parts, among them J1_+15 PIN2F061.100, J2_+15 PIN2F061.100, J3_GND PIN2F061.100, J4_GND PIN2F061.100, J5_-15 PIN2F061.100, J6_-15 PIN2F061.100, T1 TEN_60-2423N

Commit message: Add files via upload
latest power sandwitch files updated
Parts:
- removed DC_IO: 1X2-3.5MM, adafruit:1X2-3.5MM
- added DC_IN1, DC_IN2: 1X2-3.5MM, adafruit:1X2-3.5MM
- moved NOPOSREG 2.83 mm to (5.90, 51.0)
- moved IC1 2.00 mm to (-4.00, 31.0)
- moved T1 2.00 mm to (1.00, 11.0)
Connections:
- removed net N$13: IC1.3, J3_GND.A1, J3_GND.A2, J4_GND.A1, J4_GND.A2, T1.5
- new net N$1: DC_IN1.1, DC_IN2.2, IC1.3, J3_GND.A1, J3_GND.A2, J4_GND.A1, J4_GND.A2, T1.5
- net -15IN: now also DC_IN2.1
- net 15IN: now also DC_IN1.2
- net N$11: no longer DC_IO.2
- net NEGVIN: no longer DC_IO.1
Routing:
- net N$10: track 0.00 -> 106.8 mm
- net N$11: track 0.00 -> 96.2 mm
- net 15IN: track 0.00 -> 77.2 mm
- net N$1: track 0.00 -> 70.0 mm, vias 3 -> 0
- net -15IN: track 0.00 -> 65.0 mm
- net NEGVIN: track 0.00 -> 49.9 mm
Other:
- board size 16 x 60 mm -> 36.7 x 71.7 mm
- board text added: "Dual DC supply"
- board text added: "Single DC supply"
