File: Add-ons/Power Sandwitch/Power Sandwitch.sch (EAGLE design)
At the start: 13 parts, among them J1_+15 PIN2F061.100, J2_+15 PIN2F061.100, J3_GND PIN2F061.100, J4_GND PIN2F061.100, J5_-15 PIN2F061.100, J6_-15 PIN2F061.100, T1 TEN_60-2423N

Commit message: Add files via upload
latest power sandwitch files updated
Parts:
- removed DC_IO: 1X2-3.5MM, adafruit:1X2-3.5MM
- added DC_IN1, DC_IN2: 1X2-3.5MM, adafruit:1X2-3.5MM
Connections:
- removed net N$13: IC1.+VOUT, J3_GND.1, J4_GND.1, T1.COMMON
- new net N$1: DC_IN1.1, DC_IN2.2, IC1.+VOUT, J3_GND.1, J4_GND.1, T1.COMMON
- net -15IN: now also DC_IN2.1
- net 15IN: now also DC_IN1.2
- net N$11: no longer DC_IO.2
- net NEGVIN: no longer DC_IO.1
Changed lines of the file:
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@@
 <part name="IC1" library="traco_thl_tel_series" deviceset="THL_20WI_SERIES" device=""/>
 <part name="NOPOSREG" library="resistor-shunt" deviceset="SMT-REF" device=""/>
-<part name="DC_IO" library="adafruit" deviceset="1X2" device="-3.5MM"/>
 <part name="F3" library="fuse" deviceset="GSH15" device=""/>
 <part name="DC_IN" library="adafruit" deviceset="1X2" device="-3.5MM"/>
 <part name="NOFUSE" library="resistor-shunt" deviceset="SMT-REF" device=""/>
+<part name="DC_IN1" library="adafruit" deviceset="1X2" device="-3.5MM"/>
+<part name="DC_IN2" library="adafruit" deviceset="1X2" device="-3.5MM"/>
 </parts>
 <sheets>
@@
 <instance part="IC1" gate="G$1" x="162.56" y="149.86"/>
 <instance part="NOPOSREG" gate="G$1" x="139.7" y="162.56" rot="R90"/>
-<instance part="DC_IO" gate="G$1" x="114.3" y="139.7" rot="R180"/>
 <instance part="F3" gate="1" x="127" y="149.86"/>
 <instance part="DC_IN" gate="G$1" x="114.3" y="149.86" rot="R180"/>
 <instance part="NOFUSE" gate="G$1" x="127" y="157.48" rot="R180"/>
+<instance part="DC_IN1" gate="G$1" x="220.98" y="160.02" rot="R180"/>
+<instance part="DC_IN2" gate="G$1" x="220.98" y="104.14" rot="R180"/>
 </instances>
 <busses>
@@
 <junction x="233.68" y="111.76"/>
 <wire x1="233.68" y1="114.3" x2="233.68" y2="111.76" width="0.1524" layer="91"/>
-<wire x1="210.82" y1="114.3" x2="233.68" y2="114.3" width="0.1524" layer="91"/>
+<wire x1="210.82" y1="114.3" x2="231.14" y2="114.3" width="0.1524" layer="91"/>
 <junction x="210.82" y="114.3"/>
 <label x="241.3" y="109.22" size="1.778" layer="95"/>
+<wire x1="231.14" y1="114.3" x2="233.68" y2="114.3" width="0.1524" layer="91"/>
 <wire x1="233.68" y1="111.76" x2="246.38" y2="111.76" width="0.1524" layer="91"/>
 <label x="233.68" y="116.84" size="1.778" layer="95"/>
@@
 <wire x1="195.58" y1="152.4" x2="195.58" y2="116.84" width="0.1524" layer="91"/>
 <junction x="195.58" y="116.84"/>
+<pinref part="DC_IN2" gate="G$1" pin="1"/>
+<wire x1="226.06" y1="101.6" x2="231.14" y2="101.6" width="0.1524" layer="91"/>
+<wire x1="231.14" y1="101.6" x2="231.14" y2="114.3" width="0.1524" layer="91"/>
+<junction x="231.14" y="114.3"/>
 </segment>
 </net>
@@
 <pinref part="J1_+15" gate="-1" pin="1"/>
 <wire x1="210.82" y1="139.7" x2="210.82" y2="144.78" width="0.1524" layer="91"/>
-<wire x1="210.82" y1="144.78" x2="233.68" y2="144.78" width="0.1524" layer="91"/>
+<wire x1="210.82" y1="144.78" x2="231.14" y2="144.78" width="0.1524" layer="91"/>
+<wire x1="231.14" y1="144.78" x2="233.68" y2="144.78" width="0.1524" layer="91"/>
 <wire x1="233.68" y1="144.78" x2="233.68" y2="139.7" width="0.1524" layer="91"/>
 <junction x="210.82" y="144.78"/>
@@
 <wire x1="210.82" y1="167.64" x2="210.82" y2="144.78" width="0.1524" layer="91"/>
 <pinref part="NOPOSREG" gate="G$1" pin="1"/>
+<pinref part="DC_IN1" gate="G$1" pin="2"/>
+<wire x1="226.06" y1="160.02" x2="231.14" y2="160.02" width="0.1524" layer="91"/>
+<wire x1="231.14" y1="160.02" x2="231.14" y2="144.78" width="0.1524" layer="91"/>
+<junction x="231.14" y="144.78"/>
 </segment>
 </net>
@@
 <wire x1="139.7" y1="134.62" x2="127" y2="134.62" width="0.1524" layer="91"/>
 <junction x="139.7" y="134.62"/>
-<pinref part="DC_IO" gate="G$1" pin="1"/>
 <wire x1="127" y1="134.62" x2="121.92" y2="134.62" width="0.1524" layer="91"/>
-<wire x1="119.38" y1="137.16" x2="121.92" y2="137.16" width="0.1524" layer="91"/>
-<wire x1="121.92" y1="137.16" x2="121.92" y2="134.62" width="0.1524" layer="91"/>
 <pinref part="DC_IN" gate="G$1" pin="1"/>
 <wire x1="119.38" y1="147.32" x2="127" y2="147.32" width="0.1524" layer="91"/>
@@
 <junction x="127" y="134.62"/>
 <wire x1="121.92" y1="134.62" x2="121.92" y2="129.54" width="0.1524" layer="91"/>
-<junction x="121.92" y="134.62"/>
 <label x="121.92" y="129.54" size="1.778" layer="95"/>
 </segment>
@@
 <net name="N$11" class="0">
 <segment>
-<pinref part="DC_IO" gate="G$1" pin="2"/>
-<wire x1="119.38" y1="139.7" x2="121.92" y2="139.7" width="0.1524" layer="91"/>
 <pinref part="F3" gate="1" pin="1"/>
-<wire x1="121.92" y1="139.7" x2="121.92" y2="149.86" width="0.1524" layer="91"/>
 <pinref part="DC_IN" gate="G$1" pin="2"/>
 <wire x1="119.38" y1="149.86" x2="121.92" y2="149.86" width="0.1524" layer="91"/>
@@
 </segment>
 </net>
-<net name="N$13" class="0">
+<net name="N$1" class="0">
 <segment>
+<pinref part="DC_IN1" gate="G$1" pin="1"/>
+<wire x1="226.06" y1="157.48" x2="226.06" y2="129.54" width="0.1524" layer="91"/>
+<pinref part="DC_IN2" gate="G$1" pin="2"/>
 <pinref part="J3_GND" gate="-1" pin="1"/>
 <pinref part="J4_GND" gate="-1" pin="1"/>
+<wire x1="226.06" y1="129.54" x2="226.06" y2="104.14" width="0.1524" layer="91"/>
 <wire x1="210.82" y1="121.92" x2="210.82" y2="129.54" width="0.1524" layer="91"/>
 <junction x="210.82" y="129.54"/>
@@
 <pinref part="T1" gate="G$1" pin="COMMON"/>
 <wire x1="187.96" y1="124.46" x2="190.5" y2="124.46" width="0.1524" layer="91"/>
+<wire x1="226.06" y1="129.54" x2="210.82" y2="129.54" width="0.1524" layer="91"/>
+<junction x="226.06" y="129.54"/>
 </segment>
 </net>
-<net name="N$31" class="0">
-<segment>
-<wire x1="233.68" y1="129.54" x2="233.68" y2="124.46" width="0.1524" layer="91"/>
-<label x="233.68" y="132.08" size="1.778" layer="95"/>
-</segment>
-</net>
